Commit message: Fix wheel joint type

File: sagan_description/urdf/wheel/cylinder_wheel.urdf.xacro (robot description, xacro)
@@ -28,5 +28,5 @@
 			</collision>
 		</link>
-        <joint name="${wheel_prefix}_wheel_joint" type="fixed">
+        <joint name="${wheel_prefix}_wheel_joint" type="continuous">
 			<parent link="base_link"/>
 			<child link="${wheel_prefix}_wheel_link"/>
