Commit message: Add gazebo tags on URDFs and create READMEs

File: sagan_description/robots/sagan_box.urdf.xacro (robot description, xacro)
@@ -1,4 +1,5 @@
 <?xml version="1.0"?>
 <robot name="sagan_box" xmlns:xacro="http://www.ros.org/wiki/xacro">
+	<xacro:arg name="gazebo" default="true"/>
 	<!-- Include Sagan Parameters -->
 	<xacro:include filename="$(find sagan_description)/urdf/common.xacro"/>
@@ -9,19 +10,19 @@
 	<!-- Robot Definition -->
     <!-- Chassis -->
-	<xacro:box_chassis name="base_link"/>
+	<xacro:box_chassis name="base_link" gazebo="$(arg gazebo)"/>
 	<!-- FL Wheel -->
-	<xacro:cylinder_wheel wheel_prefix="fl">
+	<xacro:cylinder_wheel wheel_prefix="fl" gazebo="$(arg gazebo)">
 		<origin xyz="${wheel_x_pos} ${wheel_y_pos} ${wheel_z_pos}" rpy="${-PI/2} 0 0"/>
 	</xacro:cylinder_wheel>
 	<!-- FR Wheel -->
-	<xacro:cylinder_wheel wheel_prefix="fr">
+	<xacro:cylinder_wheel wheel_prefix="fr" gazebo="$(arg gazebo)">
 		<origin xyz="${wheel_x_pos} ${-wheel_y_pos} ${wheel_z_pos}" rpy="${PI/2} 0 0"/>
 	</xacro:cylinder_wheel>
 	<!-- BL Wheel -->
-	<xacro:cylinder_wheel wheel_prefix="bl">
+	<xacro:cylinder_wheel wheel_prefix="bl" gazebo="$(arg gazebo)">
 		<origin xyz="${-wheel_x_pos} ${wheel_y_pos} ${wheel_z_pos}" rpy="${-PI/2} 0 0"/>
 	</xacro:cylinder_wheel>
 	<!-- BR Wheel -->
-	<xacro:cylinder_wheel wheel_prefix="br">
+	<xacro:cylinder_wheel wheel_prefix="br" gazebo="$(arg gazebo)">
 		<origin xyz="${-wheel_x_pos} ${-wheel_y_pos} ${wheel_z_pos}" rpy="${PI/2} 0 0"/>
 	</xacro:cylinder_wheel>

File: sagan_description/urdf/chassis/box_chassis.urdf.xacro (robot description, xacro)
@@ -1,6 +1,8 @@
 <?xml version="1.0"?>
 <robot xmlns:xacro="http://www.ros.org/wiki/xacro">
+	<!-- Gazebo Parameters -->
+	<xacro:include filename="$(find sagan_description)/urdf/chassis/box_chassis.gazebo.xacro"/>
 	<!-- Box Chassis -->
-	<xacro:macro name="box_chassis" params="name">
+	<xacro:macro name="box_chassis" params="name gazebo">
 		<link name="${name}">
 			<inertial>
@@ -15,4 +17,7 @@
 					<box size="${chassis_x_size} ${chassis_y_size} ${chassis_z_size}"/>
 				</geometry>
+	      		<material name="">
+    				<color rgba="${175/255} ${175/255} ${175/255} 1.0"/>
+  				</material>
 			</visual>
 			<collision>
@@ -23,4 +28,7 @@
 			</collision>
 		</link>
+		<xacro:if value="${gazebo}">
+			<xacro:box_chassis_gazebo name="${name}" />
+		</xacro:if>
 	</xacro:macro>
 </robot>

File: sagan_description/urdf/wheel/cylinder_wheel.urdf.xacro (robot description, xacro)
@@ -1,6 +1,8 @@
 <?xml version="1.0"?>
 <robot xmlns:xacro="http://www.ros.org/wiki/xacro">
+	<!-- Gazebo Parameters -->
+	<xacro:include filename="$(find sagan_description)/urdf/wheel/cylinder_wheel.gazebo.xacro"/>
 	<!-- Cylinder Wheel -->
-	<xacro:macro name="cylinder_wheel" params="wheel_prefix *origin">
+	<xacro:macro name="cylinder_wheel" params="wheel_prefix *origin gazebo">
 		<link name="${wheel_prefix}_wheel_link">
 			<inertial>
@@ -16,5 +18,5 @@
 	      		</geometry>
 	      		<material name="">
-    				<color rgba="${45/255} ${45/255} ${45/255} 1.0"/>
+    				<color rgba="${0/255} ${0/255} ${0/255} 1.0"/>
   				</material>
 			</visual>
@@ -26,5 +28,5 @@
 			</collision>
 		</link>
-        <joint name="${wheel_prefix}_wheel_joint" type="continuous">
+        <joint name="${wheel_prefix}_wheel_joint" type="fixed">
 			<parent link="base_link"/>
 			<child link="${wheel_prefix}_wheel_link"/>
@@ -32,4 +34,7 @@
 			<axis xyz="0 0 -1" rpy="0 0 0" />
 		</joint>
+		<xacro:if value="${gazebo}">
+			<xacro:cylinder_wheel_gazebo wheel_prefix="${wheel_prefix}" />
+		</xacro:if>
 	</xacro:macro>
 </robot>

Commit message: Create ROS2 control pkg and setup diff_drive controller

File: sagan_description/robots/sagan_box.urdf.xacro (robot description, xacro)
@@ -8,4 +8,8 @@
 	<!-- Include Wheel Description -->
 	<xacro:include filename="$(find sagan_description)/urdf/wheel/cylinder_wheel.urdf.xacro"/>
+	<!-- Include ROS2 Control Hardware Components -->
+	<xacro:include filename="$(find sagan_description)/ros2_control/sagan_system.ros2_control.xacro"/>
+	<!-- Include Gazebo Parameters -->
+	<xacro:include filename="$(find sagan_description)/gazebo/sagan_box.gazebo.xacro"/>
 	<!-- Robot Definition -->
     <!-- Chassis -->
@@ -13,5 +17,5 @@
 	<!-- FL Wheel -->
 	<xacro:cylinder_wheel wheel_prefix="fl" gazebo="$(arg gazebo)">
-		<origin xyz="${wheel_x_pos} ${wheel_y_pos} ${wheel_z_pos}" rpy="${-PI/2} 0 0"/>
+		<origin xyz="${wheel_x_pos} ${wheel_y_pos} ${wheel_z_pos}" rpy="${PI/2} 0 0"/>
 	</xacro:cylinder_wheel>
 	<!-- FR Wheel -->
@@ -21,5 +25,5 @@
 	<!-- BL Wheel -->
 	<xacro:cylinder_wheel wheel_prefix="bl" gazebo="$(arg gazebo)">
-		<origin xyz="${-wheel_x_pos} ${wheel_y_pos} ${wheel_z_pos}" rpy="${-PI/2} 0 0"/>
+		<origin xyz="${-wheel_x_pos} ${wheel_y_pos} ${wheel_z_pos}" rpy="${PI/2} 0 0"/>
 	</xacro:cylinder_wheel>
 	<!-- BR Wheel -->
@@ -27,3 +31,7 @@
 		<origin xyz="${-wheel_x_pos} ${-wheel_y_pos} ${wheel_z_pos}" rpy="${PI/2} 0 0"/>
 	</xacro:cylinder_wheel>
+	<!-- ROS2 Control Componentes -->
+	<xacro:sagan_system name="sagan_system_interfaces" gazebo="$(arg gazebo)"/>
+	<!-- Gazebo -->
+	<xacro:sagan_gazebo name="sagan_gazebo" />
 </robot>

Commit message: Rename xacro argument gazebo to sim_gazebo

File: sagan_description/robots/sagan_box.urdf.xacro (robot description, xacro)
@@ -11,27 +11,31 @@
 	<xacro:include filename="$(find sagan_description)/ros2_control/sagan_system.ros2_control.xacro"/>
 	<!-- Include Gazebo Parameters -->
-	<xacro:include filename="$(find sagan_description)/gazebo/sagan_box.gazebo.xacro"/>
+	<xacro:if value="$(arg sim_gazebo)">
+		<xacro:include filename="$(find sagan_description)/gazebo/sagan_box.gazebo.xacro"/>
+	</xacro:if>
 	<!-- Robot Definition -->
     <!-- Chassis -->
-	<xacro:box_chassis name="base_link" gazebo="$(arg gazebo)"/>
+	<xacro:box_chassis name="base_link" sim_gazebo="$(arg sim_gazebo)"/>
 	<!-- FL Wheel -->
-	<xacro:cylinder_wheel wheel_prefix="fl" gazebo="$(arg gazebo)">
+	<xacro:cylinder_wheel wheel_prefix="fl" sim_gazebo="$(arg sim_gazebo)">
 		<origin xyz="${wheel_x_pos} ${wheel_y_pos} ${wheel_z_pos}" rpy="${PI/2} 0 0"/>
 	</xacro:cylinder_wheel>
 	<!-- FR Wheel -->
-	<xacro:cylinder_wheel wheel_prefix="fr" gazebo="$(arg gazebo)">
+	<xacro:cylinder_wheel wheel_prefix="fr" sim_gazebo="$(arg sim_gazebo)">
 		<origin xyz="${wheel_x_pos} ${-wheel_y_pos} ${wheel_z_pos}" rpy="${PI/2} 0 0"/>
 	</xacro:cylinder_wheel>
 	<!-- BL Wheel -->
-	<xacro:cylinder_wheel wheel_prefix="bl" gazebo="$(arg gazebo)">
+	<xacro:cylinder_wheel wheel_prefix="bl" sim_gazebo="$(arg sim_gazebo)">
 		<origin xyz="${-wheel_x_pos} ${wheel_y_pos} ${wheel_z_pos}" rpy="${PI/2} 0 0"/>
 	</xacro:cylinder_wheel>
 	<!-- BR Wheel -->
-	<xacro:cylinder_wheel wheel_prefix="br" gazebo="$(arg gazebo)">
+	<xacro:cylinder_wheel wheel_prefix="br" sim_gazebo="$(arg sim_gazebo)">
 		<origin xyz="${-wheel_x_pos} ${-wheel_y_pos} ${wheel_z_pos}" rpy="${PI/2} 0 0"/>
 	</xacro:cylinder_wheel>
 	<!-- ROS2 Control Componentes -->
-	<xacro:sagan_system name="sagan_system_interfaces" gazebo="$(arg gazebo)"/>
+	<xacro:sagan_system name="sagan_system_interfaces" sim_gazebo="$(arg sim_gazebo)"/>
 	<!-- Gazebo -->
-	<xacro:sagan_gazebo name="sagan_gazebo" />
+	<xacro:if value="$(arg sim_gazebo)">
+		<xacro:sagan_gazebo name="sagan_gazebo" />
+	</xacro:if>
 </robot>

File: sagan_description/ros2_control/sagan_system.ros2_control.xacro (robot description, xacro)
@@ -1,7 +1,7 @@
 <?xml version="1.0"?>
 <robot xmlns:xacro="http://www.ros.org/wiki/xacro">
-    <xacro:macro name="sagan_system" params="name gazebo">
+    <xacro:macro name="sagan_system" params="name sim_gazebo">
         <ros2_control name="GazeboSystem" type="system">
-            <xacro:if value="${gazebo}">
+            <xacro:if value="${sim_gazebo}">
                 <hardware>
                     <plugin>gazebo_ros2_control/GazeboSystem</plugin>

File: sagan_description/urdf/chassis/box_chassis.urdf.xacro (robot description, xacro)
@@ -4,5 +4,5 @@
 	<xacro:include filename="$(find sagan_description)/urdf/chassis/box_chassis.gazebo.xacro"/>
 	<!-- Box Chassis -->
-	<xacro:macro name="box_chassis" params="name gazebo">
+	<xacro:macro name="box_chassis" params="name sim_gazebo">
 		<link name="${name}">
 			<inertial>
@@ -28,5 +28,5 @@
 			</collision>
 		</link>
-		<xacro:if value="${gazebo}">
+		<xacro:if value="${sim_gazebo}">
 			<xacro:box_chassis_gazebo name="${name}" />
 		</xacro:if>

File: sagan_description/urdf/wheel/cylinder_wheel.urdf.xacro (robot description, xacro)
@@ -4,5 +4,5 @@
 	<xacro:include filename="$(find sagan_description)/urdf/wheel/cylinder_wheel.gazebo.xacro"/>
 	<!-- Cylinder Wheel -->
-	<xacro:macro name="cylinder_wheel" params="wheel_prefix *origin gazebo">
+	<xacro:macro name="cylinder_wheel" params="wheel_prefix *origin sim_gazebo">
 		<link name="${wheel_prefix}_wheel_link">
 			<inertial>
@@ -34,5 +34,5 @@
 			<axis xyz="0 0 -1" rpy="0 0 0" />
 		</joint>
-		<xacro:if value="${gazebo}">
+		<xacro:if value="${sim_gazebo}">
 			<xacro:cylinder_wheel_gazebo wheel_prefix="${wheel_prefix}" />
 		</xacro:if>
