Commit message: Update mass and inertia values from Husky robot

File: sagan_description/urdf/common.xacro (robot description, xacro)
@@ -6,5 +6,5 @@
 	<xacro:property name="chassis_y_com" value="0.0"/>
 	<xacro:property name="chassis_z_com" value="0.0"/>
-	<xacro:property name="chassis_mass" value="10.0"/>
+	<xacro:property name="chassis_mass" value="46.034"/>
 	<xacro:property name="chassis_ixx" value="0.6022"/>
 	<xacro:property name="chassis_iyy" value="1.7386"/>
@@ -20,8 +20,8 @@
 	<xacro:property name="wheel_y_com" value="0.0"/>
 	<xacro:property name="wheel_z_com" value="0.0"/>
-	<xacro:property name="wheel_mass" value="0.5"/>
-	<xacro:property name="wheel_ixx" value="0.01"/>
-	<xacro:property name="wheel_iyy" value="0.01"/>
-	<xacro:property name="wheel_izz" value="0.01"/>
+	<xacro:property name="wheel_mass" value="2.637"/>
+	<xacro:property name="wheel_ixx" value="0.02467"/>
+	<xacro:property name="wheel_iyy" value="0.02467"/>
+	<xacro:property name="wheel_izz" value="0.04411"/>
 	<xacro:property name="wheel_ixy" value="0.0"/>
 	<xacro:property name="wheel_ixz" value="0.0"/>

File: sagan_description/urdf/wheel/cylinder_wheel.gazebo.xacro (robot description, xacro)
@@ -4,11 +4,9 @@
 		<!-- Wheel Link -->
 		<gazebo reference="${wheel_prefix}_wheel_link">
-			<mu1>10</mu1>
-			<mu2>10</mu2>
-			<kp>500000.0</kp>
-			<kd>10.0</kd>
-			<minDepth>0.001</minDepth>
-			<maxVel>0.1</maxVel>
-			<fdir1>1 0 0</fdir1>
+			<mu1 value="2.0"/>
+			<mu2 value="0.1"/>
+			<kp value="10000000.0" />
+			<kd value="1.0" />
+			<fdir1 value="1 0 0"/>
 			<material>Gazebo/FlatBlack</material>
 		</gazebo>
